File: USB_C_Trig_Board_Simple_Multi_Layer/USB_C_Simple_Trig_Multi_Layer/USB_C_Simple_Trig.kicad_pcb (KiCad board)
At the start: 6 copper layers, 45.9 x 48.7 mm, 49 parts, among them IC1 AP33772SDKZ-13-FA01, J1 USB_C_Receptacle, J2 Screw_Terminal_01x04, J3 Conn_01x06_Pin, J4 Conn_ARM_JTAG_SWD_10, Q1 BUK7880-55A/CUX, Q2 BUK7880-55A/CUX, SW1 SW_Push, U10 AP2127N-3.3, U5 STM32C011F6Px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

Commit message: Silkscreen update for both simple trig boards.
Other:
- board text added: "USB-C PD Simple Trigger Board V1.0 Up to 28V 5A with PD EPR PD PPS compatible 6-layer board hi@ihsan.cc"
- board text removed: "USB-C PD Simple Trigger Board V1.0 Up to 28V 5A with PD EPR PD PPS compatible hi@ihsan.cc"
Changed lines of the file:
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@@
 		)
 	)
-	(gr_text "USB-C PD Simple Trigger Board V1.0\nUp to 28V 5A with PD EPR\nPD PPS compatible\n\nhi@ihsan.cc\n"
-		(at 130.65 84.55 270)
+	(gr_text "USB-C PD Simple Trigger Board V1.0\nUp to 28V 5A with PD EPR\nPD PPS compatible\n6-layer board\n\nhi@ihsan.cc\n"
+		(at 129.5 84.5 270)
 		(layer "B.SilkS")
 		(effects
